File: hardware/boards/v0.1/memory.kicad_sch (KiCad schematic)
At the start: 12 parts, among them IC1 W25Q512JVEIQ, IC4 IS42S16160J-7TLI, J3 MICRO_SD, U22 XTSDG08GWSIGA

Commit message: feat: more BOM selection
Parts:
- added TP29: PICO, TestPoint:TestPoint_Pad_D1.0mm, symbol Connector:TestPoint
- added TP41: CLK, TestPoint:TestPoint_Pad_D1.0mm, symbol Connector:TestPoint
- added TP42: POCI, TestPoint:TestPoint_Pad_D1.0mm, symbol Connector:TestPoint
- added TP43: XTSDG_CS, TestPoint:TestPoint_Pad_D1.0mm, symbol Connector:TestPoint
- added TP44: SD_CS, TestPoint:TestPoint_Pad_D1.0mm, symbol Connector:TestPoint
Connections:
- net SD_CS: now also TP44.1
- net SPI.CLK: now also TP41.1
- net SPI.PICO: now also TP29.1
- net SPI.POCI: now also TP42.1
- net XTSDG_CS: now also TP43.1

Commit message: feat: swap out of stock components
Parts:
- IC1: Manufacturer_Name Winbond -> (none); Manufacturer_Part_Number W25Q512JVEIQ -> (none)
- IC4: Manufacturer_Name Integrated Silicon Solution Inc. -> (none); Manufacturer_Part_Number IS42S16160J-7TLI -> (none)
Changed lines of the file:
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@@
+		(polyline
+			(pts
+				(xy 121.92 81.28) (xy 121.92 101.6) (xy 134.62 101.6) (xy 134.62 81.28)
+			)
+			(stroke
+				(width 0)
+				(type dash)
+			)
+			(fill
+				(type none)
+			)
+		)
+	)
+	(rule_area
 		(polyline
 			(pts
 				(xy 121.92 81.28) (xy 121.92 59.69) (xy 134.62 59.69) (xy 134.62 81.28)
-			)
-			(stroke
-				(width 0)
-				(type dash)
-			)
-			(fill
-				(type none)
-			)
-		)
-	)
-	(rule_area
-		(polyline
-			(pts
-				(xy 121.92 81.28) (xy 121.92 101.6) (xy 134.62 101.6) (xy 134.62 81.28)
 			)
 			(stroke
@@
 			)
 		)
-		(property "Manufacturer_Name" "Winbond"
-			(at 288.29 736.83 0)
-			(effects
-				(font
-					(size 1.27 1.27)
-				)
-				(justify left top)
-				(hide yes)
-			)
-		)
-		(property "Manufacturer_Part_Number" "W25Q512JVEIQ"
-			(at 288.29 836.83 0)
-			(effects
-				(font
-					(size 1.27 1.27)
-				)
-				(justify left top)
-				(hide yes)
-			)
-		)
 		(property "JLC" "C2986165"
 			(at 269.24 48.26 0)
@@
 			(effects
 				(font
-					(size 1.27 1.27)
-				)
-				(justify left top)
-				(hide yes)
-			)
-		)
-		(property "Manufacturer_Name" "Integrated Silicon Solution Inc."
-			(at 118.11 758.42 0)
-			(effects
-				(font
-					(size 1.27 1.27)
-				)
-				(justify left top)
-				(hide yes)
-			)
-		)
-		(property "Manufacturer_Part_Number" "IS42S16160J-7TLI"
-			(at 118.11 858.42 0)
-			(effects
-				(font

Commit message: chore: schematic cleanup
Parts:
- C64: value 0.1uF -> 100nF; JLC C15525 -> C1525
Changed lines of the file:
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@@
 			)
 		)
-		(property "Value" "0.1uF"
+		(property "Value" "100nF"
 			(at 215.646 30.734 0)
 			(effects
@@
 			)
 		)
-		(property "JLC" "C15525"
+		(property "JLC" "C1525"
 			(at 214.63 27.94 0)
 			(effects
