File: hardware/boards/v0.1/keypad.kicad_sch (KiCad schematic)
At the start: 78 parts, among them SW1 TRIG1, SW10 TRIG10, SW11 TRIG11, SW12 TRIG12, SW13 TRIG13, SW14 TRIG14, SW15 TRIG15, SW16 TRIG16, SW17 MENU0, SW19 MENU1, SW2 TRIG2, SW20 MENU2, SW21 MENU3, SW3 TRIG3, SW4 TRIG4, SW5 TRIG5, SW6 TRIG6, SW7 TRIG7, SW8 TRIG8, SW9 TRIG9, U25 TCA8418RTWR, U38 ADS7128IRTER

Commit message: feat: swap out of stock components
Parts:
- D1, D10, D11, D12, D13, D14, D15, D16, D2, D22, D23, D24, D25, D26, D27, D28, D29, D3, D30, D31, D32, D33, D34, D35, D36, D37, D4, D5, D6, D7, D8, D9: footprint Diode_SMD:D_SOD-123 -> Diode_SMD:D_SOD-323
Changed lines of the file:
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@@
 			)
 		)
-		(property "Footprint" "Diode_SMD:D_SOD-123"
+		(property "Footprint" "Diode_SMD:D_SOD-323"
 			(at 179.07 35.56 0)
 			(effects
@@
 			)
 		)
-		(property "Footprint" "Diode_SMD:D_SOD-123"
+		(property "Footprint" "Diode_SMD:D_SOD-323"
 			(at 224.79 127 0)
 			(effects
@@
 			)
 		)
-		(property "Footprint" "Diode_SMD:D_SOD-123"
+		(property "Footprint" "Diode_SMD:D_SOD-323"
 			(at 152.4 127 0)
 			(effects
@@
 			)
 		)
-		(property "Footprint" "Diode_SMD:D_SOD-123"
+		(property "Footprint" "Diode_SMD:D_SOD-323"
 			(at 204.47 50.8 0)
 			(effects
@@
 			)
 		)
-		(property "Footprint" "Diode_SMD:D_SOD-123"
+		(property "Footprint" "Diode_SMD:D_SOD-323"
 			(at 176.53 111.76 0)
 			(effects
@@
 			)
 		)
-		(property "Footprint" "Diode_SMD:D_SOD-123"
+		(property "Footprint" "Diode_SMD:D_SOD-323"
 			(at 229.87 66.04 0)
 			(effects
@@
 			)
 		)
-		(property "Footprint" "Diode_SMD:D_SOD-123"
+		(property "Footprint" "Diode_SMD:D_SOD-323"
 			(at 153.67 35.56 0)
 			(effects
@@
 			)
 		)
-		(property "Footprint" "Diode_SMD:D_SOD-123"
+		(property "Footprint" "Diode_SMD:D_SOD-323"
 			(at 200.66 142.24 0)
 			(effects
@@
 			)
 		)
-		(property "Footprint" "Diode_SMD:D_SOD-123"
+		(property "Footprint" "Diode_SMD:D_SOD-323"
 			(at 200.66 111.76 0)
 			(effects
@@
 			)
 		)
-		(property "Footprint" "Diode_SMD:D_SOD-123"
+		(property "Footprint" "Diode_SMD:D_SOD-323"
 			(at 179.07 50.8 0)
 			(effects
@@
 			)
 		)
-		(property "Footprint" "Diode_SMD:D_SOD-123"
+		(property "Footprint" "Diode_SMD:D_SOD-323"
 			(at 179.07 81.28 0)
 			(effects
@@
 			)
 		)
-		(property "Footprint" "Diode_SMD:D_SOD-123"
+		(property "Footprint" "Diode_SMD:D_SOD-323"
 			(at 153.67 81.28 0)
 			(effects
@@
 			)
 		)
-		(property "Footprint" "Diode_SMD:D_SOD-123"
+		(property "Footprint" "Diode_SMD:D_SOD-323"
 			(at 224.79 157.48 0)
 			(effects
@@
 			)
 		)
-		(property "Footprint" "Diode_SMD:D_SOD-123"
+		(property "Footprint" "Diode_SMD:D_SOD-323"
 			(at 224.79 142.24 0)
 			(effects
@@
 			)
 		)
-		(property "Footprint" "Diode_SMD:D_SOD-123"
+		(property "Footprint" "Diode_SMD:D_SOD-323"
 			(at 152.4 142.24 0)
 			(effects
@@
 			)
 		)
-		(property "Footprint" "Diode_SMD:D_SOD-123"
+		(property "Footprint" "Diode_SMD:D_SOD-323"
 			(at 204.47 35.56 0)
 			(effects
@@
 			)
 		)
-		(property "Footprint" "Diode_SMD:D_SOD-123"
+		(property "Footprint" "Diode_SMD:D_SOD-323"
 			(at 152.4 111.76 0)
 			(effects
@@
 			)
 		)
-		(property "Footprint" "Diode_SMD:D_SOD-123"
+		(property "Footprint" "Diode_SMD:D_SOD-323"
 			(at 152.4 157.48 0)
 			(effects
@@
 			)
 		)
-		(property "Footprint" "Diode_SMD:D_SOD-123"
+		(property "Footprint" "Diode_SMD:D_SOD-323"
 			(at 204.47 66.04 0)
 			(effects
@@
 			)
 		)
-		(property "Footprint" "Diode_SMD:D_SOD-123"
+		(property "Footprint" "Diode_SMD:D_SOD-323"
 			(at 204.47 81.28 0)
 			(effects
@@
 			)
 		)
-		(property "Manufacturer_Name" ""
-			(at 67.31 105.41 0)
-			(effects
-				(font
-					(size 1.27 1.27)
-				)
-			)
-		)
-		(property "Manufacturer_Part_Number" ""
-			(at 67.31 105.41 0)
-			(effects
-				(font
-					(size 1.27 1.27)
-				)
-			)
-		)
 		(property "MANUFACTURER" ""
 			(at 67.31 105.41 0)
@@
 			)
 		)
-		(property "Footprint" "Diode_SMD:D_SOD-123"
+		(property "Footprint" "Diode_SMD:D_SOD-323"
 			(at 200.66 127 0)
 			(effects
@@
 			)
 		)
-		(property "Footprint" "Diode_SMD:D_SOD-123"
+		(property "Footprint" "Diode_SMD:D_SOD-323"
 			(at 229.87 50.8 0)
 			(effects
@@
 			)
 		)
-		(property "Manufacturer_Name" ""
-			(at 80.01 105.41 0)
-			(effects
-				(font
-					(size 1.27 1.27)
-				)
-			)
-		)
-		(property "Manufacturer_Part_Number" ""
-			(at 80.01 105.41 0)
-			(effects
-				(font
-					(size 1.27 1.27)
-				)
-			)
-		)
 		(property "MANUFACTURER" ""
 			(at 80.01 105.41 0)
@@
 			)
 		)
-		(property "Manufacturer_Name" ""
-			(at 46.99 149.86 0)
-			(effects
-				(font
-					(size 1.27 1.27)
-				)
-			)
-		)
-		(property "Manufacturer_Part_Number" ""
-			(at 46.99 149.86 0)
-			(effects
-				(font
-					(size 1.27 1.27)
-				)
-			)
-		)
 		(property "MANUFACTURER" ""
 			(at 46.99 149.86 0)
@@
 			)
 		)
-		(property "Footprint" "Diode_SMD:D_SOD-123"
+		(property "Footprint" "Diode_SMD:D_SOD-323"
 			(at 229.87 35.56 0)
 			(effects
@@
 			)
 		)
-		(property "Footprint" "Diode_SMD:D_SOD-123"
+		(property "Footprint" "Diode_SMD:D_SOD-323"
 			(at 224.79 111.76 0)
 			(effects
@@
 			)
 		)
-		(property "Footprint" "Diode_SMD:D_SOD-123"
+		(property "Footprint" "Diode_SMD:D_SOD-323"
 			(at 153.67 50.8 0)
 			(effects
@@
 			)
 		)
-		(property "Footprint" "Diode_SMD:D_SOD-123"
+		(property "Footprint" "Diode_SMD:D_SOD-323"
 			(at 153.67 66.04 0)
 			(effects
@@
 			)
 		)
-		(property "Footprint" "Diode_SMD:D_SOD-123"
+		(property "Footprint" "Diode_SMD:D_SOD-323"
 			(at 176.53 157.48 0)
 			(effects
@@
 			)
 		)
-		(property "Footprint" "Diode_SMD:D_SOD-123"
+		(property "Footprint" "Diode_SMD:D_SOD-323"
 			(at 229.87 81.28 0)
 			(effects
@@
 			)
 		)
-		(property "Footprint" "Diode_SMD:D_SOD-123"
+		(property "Footprint" "Diode_SMD:D_SOD-323"
 			(at 200.66 157.48 0)
 			(effects
@@
 			)
 		)
-		(property "Footprint" "Diode_SMD:D_SOD-123"
+		(property "Footprint" "Diode_SMD:D_SOD-323"
 			(at 176.53 127 0)
 			(effects
@@
 			)
 		)
-		(property "Footprint" "Diode_SMD:D_SOD-123"
+		(property "Footprint" "Diode_SMD:D_SOD-323"
 			(at 176.53 142.24 0)
 			(effects
@@
 			)
 		)
-		(property "Footprint" "Diode_SMD:D_SOD-123"
+		(property "Footprint" "Diode_SMD:D_SOD-323"
 			(at 179.07 66.04 0)
 			(effects

Commit message: chore: schematic cleanup
Parts:
- D1, D10, D11, D12, D13, D14, D15, D16, D2, D22, D23, D24, D25, D26, D27, D28, D29, D3, D30, D31, D32, D33, D34, D35, D36, D37, D4, D5, D6, D7, D8, D9: value D -> 1N4148WS
Changed lines of the file:
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@@
 			)
 		)
-		(property "Value" "D"
+		(property "Value" "1N4148WS"
 			(at 179.07 38.354 0)
 			(effects
@@
 			)
 		)
-		(property "Value" "D"
+		(property "Value" "1N4148WS"
 			(at 224.79 129.794 0)
 			(effects
@@
 			)
 		)
-		(property "Value" "D"
+		(property "Value" "1N4148WS"
 			(at 152.4 129.794 0)
 			(effects
@@
 			)
 		)
-		(property "Value" "D"
+		(property "Value" "1N4148WS"
 			(at 204.47 53.594 0)
 			(effects
@@
 			)
 		)
-		(property "Value" "D"
+		(property "Value" "1N4148WS"
 			(at 176.53 114.554 0)
 			(effects
@@
 			)
 		)
-		(property "Value" "D"
+		(property "Value" "1N4148WS"
 			(at 229.87 68.834 0)
 			(effects
@@
 			)
 		)
-		(property "Value" "D"
+		(property "Value" "1N4148WS"
 			(at 153.67 38.354 0)
 			(effects
@@
 			)
 		)
-		(property "Value" "D"
+		(property "Value" "1N4148WS"
 			(at 200.66 145.034 0)
 			(effects
@@
 			)
 		)
-		(property "Value" "D"
+		(property "Value" "1N4148WS"
 			(at 200.66 114.554 0)
 			(effects
@@
 			)
 		)
-		(property "Value" "D"
+		(property "Value" "1N4148WS"
 			(at 179.07 53.594 0)
 			(effects
@@
 			)
 		)
-		(property "Value" "D"
+		(property "Value" "1N4148WS"
 			(at 179.07 84.074 0)
 			(effects
@@
 			)
 		)
-		(property "Value" "D"
+		(property "Value" "1N4148WS"
 			(at 153.67 84.074 0)
 			(effects
@@
 			)
 		)
-		(property "Value" "D"
+		(property "Value" "1N4148WS"
 			(at 224.79 160.274 0)
 			(effects
@@
 			)
 		)
-		(property "Value" "D"
+		(property "Value" "1N4148WS"
 			(at 224.79 145.034 0)
 			(effects
@@
 			)
 		)
-		(property "Value" "D"
+		(property "Value" "1N4148WS"
 			(at 152.4 145.034 0)
 			(effects
@@
 			)
 		)
-		(property "Value" "D"
+		(property "Value" "1N4148WS"
 			(at 204.47 38.354 0)
 			(effects
@@
 			)
 		)
-		(property "Value" "D"
+		(property "Value" "1N4148WS"
 			(at 152.4 114.554 0)
 			(effects
@@
 			)
 		)
-		(property "Value" "D"
+		(property "Value" "1N4148WS"
 			(at 152.4 160.274 0)
 			(effects
@@
 			)
 		)
-		(property "Value" "D"
+		(property "Value" "1N4148WS"
 			(at 204.47 68.834 0)
 			(effects
@@
 			)
 		)
-		(property "Value" "D"
+		(property "Value" "1N4148WS"
 			(at 204.47 84.074 0)
 			(effects
@@
 			)
 		)
-		(property "Value" "D"
+		(property "Value" "1N4148WS"
 			(at 200.66 129.794 0)
 			(effects
@@
 			)
 		)
-		(property "Value" "D"
+		(property "Value" "1N4148WS"
 			(at 229.87 53.594 0)
 			(effects
@@
 			)
 		)
-		(property "Value" "D"
+		(property "Value" "1N4148WS"
 			(at 229.87 38.354 0)
 			(effects
@@
 			)
 		)
-		(property "Value" "D"
+		(property "Value" "1N4148WS"
 			(at 224.79 114.554 0)
 			(effects
@@
 			)
 		)
-		(property "Value" "D"
+		(property "Value" "1N4148WS"
 			(at 153.67 53.594 0)
 			(effects
@@
 			)
 		)
-		(property "Value" "D"
+		(property "Value" "1N4148WS"
 			(at 153.67 68.834 0)
 			(effects
@@
 			)
 		)
-		(property "Value" "D"
+		(property "Value" "1N4148WS"
 			(at 176.53 160.274 0)
 			(effects
@@
 			)
 		)
-		(property "Value" "D"
+		(property "Value" "1N4148WS"
 			(at 229.87 84.074 0)
 			(effects
@@
 			)
 		)
-		(property "Value" "D"
+		(property "Value" "1N4148WS"
 			(at 200.66 160.274 0)
 			(effects
@@
 			)
 		)
-		(property "Value" "D"
+		(property "Value" "1N4148WS"
 			(at 176.53 129.794 0)
 			(effects
@@
 			)
 		)
-		(property "Value" "D"
+		(property "Value" "1N4148WS"
 			(at 176.53 145.034 0)
 			(effects
@@
 			)
 		)
-		(property "Value" "D"
+		(property "Value" "1N4148WS"
 			(at 179.07 68.834 0)
 			(effects

Commit message: feat: change charger, fuel gauge, and battery connector, re-route power system
Parts:
- C93, C94, C95: JLC C14445 -> C52923
- R18: JLC C25531 -> C25744
Changed lines of the file:
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@@
 			)
 		)
-		(property "JLC" "C25531"
+		(property "JLC" "C25744"
 			(at 57.15 29.21 0)
 			(effects
@@
 			)
 		)
-		(property "JLC" "C14445"
+		(property "JLC" "C52923"
 			(at 67.31 105.41 0)
 			(effects
@@
 			)
 		)
-		(property "JLC" "C14445"
+		(property "JLC" "C52923"
 			(at 80.01 105.41 0)
 			(effects
@@
 			)
 		)
-		(property "JLC" "C14445"
+		(property "JLC" "C52923"
 			(at 46.99 149.86 0)
 			(effects
