File: hardware/boards/v0.1/midi_cv.kicad_sch (KiCad schematic)
At the start: 16 parts, among them J10 MIDI_OUT/THRU, J11 MIDI_IN, U19 TLP2362TPR_E

Commit message: fix: rotation offsets and LEDs on wrong side of board
Parts:
- U19: FT Rotation Offset (none) -> -90
