File: hardware/boards/v0.2/pocket_synth_v0.2/pocket_synth_v0.2.kicad_sch (KiCad schematic)
At the start: 60 parts, among them J1 Conn_ARM_JTAG_SWD_10, J10 Conn_01x05_Pin, J11 Conn_01x02_Pin, J12 Conn_01x03_Pin, J13 INPUT, J14 UART4, J2 USB, J3 AudioJack3, J4 AudioJack3, J5 AudioJack3, J6 AudioJack3, J7 DISPLAY, J8 Micro_SD_Card_Det2, J9 USART4, SW1 SW_Push, SW2 SW_Push, SW3 SW_Push, SW4 SW_Push, U1 STM32H743XIHx, U3 SDRAM, U4 STM32H753VIHx, U5 W25Q128JVS, Y1 32.768kHz, Y2 HSE

Commit message: add NINA-W13 Wifi module and BM83 Bluetooth Audio
Parts:
- removed J9: USART4, Connector_PinHeader_1.00mm:PinHeader_1x04_P1.00mm_Vertical, symbol Connector:Conn_01x04_Pin
- added D1: LED1, symbol Device:LED_Small
- added D2: LED2, symbol Device:LED_Small
- added R4, R5: R, Resistor_SMD:R_0603_1608Metric, symbol Device:R
- added U2: NORA-W40, Northernpaws_RF:NORA-W40, symbol Northernpaws_RF:NORA-W40
- added U6: Microchip_BM83, RF_Module:Microchip_BM83, symbol RF_Bluetooth:Microchip_BM83
- added U7: NINA-W13, Northernpaws_RF:ublox-NINA-W13, symbol Northernpaws_RF:ubox-NINA-W13
- J8: value Micro_SD_Card_Det2 -> SDCARD
Connections:
- net +3.3V: now also U5.8 (VCC), U2.A7 (VCCIO), U2.A8 (VCC), U2.B7 (VCCIO), U6.23 (BAT_IN), U7.10 (VCC), U7.9 (VCC_IO)
- net GND: now also J8.6 (VSS), R4.2, R5.2, U2.A1 (GND), U2.A9 (GND), U2.B2 (GND), U2.B8 (GND), U2.E4 (GND), U2.E5 (GND), U2.F4 (GND), U2.F5 (GND), U2.K2 (GND), U2.K3 (GND), U2.K5 (GND), U2.K7 (GND), U2.K8 (GND), U2.L1 (GND), U2.L9 (GND), U2.M1 (GND), U2.M2 (GND), U2.M8 (GND), U2.M9 (GND), U6.16 (GND), U6.50 (GND), U6.56 (GND), U6.57 (GND), U7.12 (GND), U7.14 (GND), U7.26 (GND), U7.30 (GND), U7.37 (GND), U7.38 (GND), U7.39 (GND), U7.40 (GND), U7.41 (GND), U7.42 (GND), U7.43 (GND), U7.44 (GND), U7.45 (GND), U7.46 (GND), U7.47 (GND), U7.48 (GND), U7.6 (GND)
- net LCD_CLK: now also U1.F16 (PG7); no longer U1.H3 (PI14)
- net SAI1_FS_A: now also U6.2 (RFS1)
- net SAI1_SCK_A: now also U6.3 (SCLK1)
- net SAI1_SD_A: now also U6.1 (DR1)
- net USART1_TX: now reaches U1.D15 (PA9)
- net USART1_TX: now also U2.B4 (GPIO6/MTCK), U6.29 (P8_6/UART_RXD), U7.23 (UART_RXD)
- net USART1_RX: now reaches U1.D14 (PA10)
- net USART1_RX: now also U2.A3 (GPIO7/MTDO), U6.30 (P8_5/UART_TXD), U7.22 (UART_TXD)
- net USART1_CTS: now reaches U1.E17 (PA11)
- net USART1_CTS: now also U2.H2 (MTMS/GPIO4), U6.31 (P3_4/UART_RTS), U7.20 (UART_RTS/RMII_TXD1)
- net USART1_RTS: now reaches U1.E16 (PA12)
- net USART1_RTS: now also U2.H1 (MTDI/GPIO5), U6.48 (P3_7/UART_CTS), U7.21 (UART_CTS/RMII_TXD0)
- new net: U2.A4 (NC), U2.A6 (NC), U2.B5 (NC), U2.B9 (NC), U2.C4 (NC), U2.C5 (NC), U2.D1 (NC), U2.D2 (NC), U2.D7 (NC), U2.E1 (NC), U2.E2 (NC), U2.E3 (NC), U2.E7 (NC), U2.F1 (NC), U2.F2 (NC), U2.F3 (NC), U2.G2 (NC), U2.G3 (NC), U2.G4 (NC), U2.G5 (NC), U2.G7 (NC), U2.H3 (NC), U2.H7 (NC), U2.J1 (NC), U2.J4 (NC), U2.J5 (NC), U2.J7 (NC), U2.K1 (NC)
- new net: U2.F7 (PBOOT/GPIO9), U2.H8 (PBOOT/GPIO9)
- new net: U7.11 (NC), U7.15 (NC), U7.33 (NC)
- new net: R5.1, U7.19 (~{RESET})
- new net: D1.1 (K), U6.32 (LED1)
- new net: D1.2 (A), D2.2 (A), U6.24 (SYS_PWR)
- new net: R4.1, U6.43 (~{RST})
- new net: D2.1 (K), U6.34 (LED2)
- no-connect marks 18 -> 39
Other:
- note added: "ESP32-C6 has UART1 for AT commands mapped by default: GPIO6 (RX) GPIO7 (TX) GPIO5 (CTS) GPIO4 (RTS)"
- note added: "ESP32-C6 uses UART0 on 16/17 for programming."
- note added: "For download mode: GPIO8=1 GPIO9=0"
- note added: "MFB is used to control the module wake/sleep mode"
- note added: "P0_0 can be used to wake the MCU when Bluetooth traffic occures."
- note added: "Pull-down holds module in reset until the MCU is ready."
- note added: "https://docs.espressif.com/projects/esp-at/en/latest/esp32c6/Get_Started/Downloading_guide.html"
- moved on the sheet: H1, H2
